File: master_node/master_node.kicad_pcb (KiCad board)
At the start: 2 copper layers, 139.7 x 137.8 mm, 33 parts, among them J1 X_Stepper, J10 A1_Encoder, J11 A2_Encoder, J12 R_Encoder, J13 XT60-in, J14 X_Power, J15 Y _Power, J16 Z_Power, J17 A1_Power, J18 A2_Power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

Commit message: too late, I am done
Parts:
- removed REF** (x4): MountingHole_5.3mm_M5_ISO7380, MountingHole:MountingHole_5.3mm_M5_ISO7380
- added H1: MountingHole, MountingHole:MountingHole_5.3mm_M5_DIN965, F.Cu at (68.6, 63.5)
- added H2: MountingHole, MountingHole:MountingHole_5.3mm_M5_DIN965, F.Cu at (68.6, 180.3)
- added H3: MountingHole, MountingHole:MountingHole_5.3mm_M5_DIN965, F.Cu at (188.0, 180.3)
- added H4: MountingHole, MountingHole:MountingHole_5.3mm_M5_DIN965, F.Cu at (188.0, 62.9)
- added J20: X_Home_SW, Connector_PinHeader_2.54mm:PinHeader_1x02_P2.54mm_Vertical, F.Cu at (178.4, 79.4)
- added J21: Y_Home_SW, Connector_PinHeader_2.54mm:PinHeader_1x02_P2.54mm_Vertical, F.Cu at (178.4, 102.2)
- added J22: Z_Home_SW, Connector_PinHeader_2.54mm:PinHeader_1x02_P2.54mm_Vertical, F.Cu at (178.4, 125.1)
- added J23: A1_Home_SW, Connector_PinHeader_2.54mm:PinHeader_1x02_P2.54mm_Vertical, F.Cu at (178.4, 90.8)
- added J24: A2_Home_SW, Connector_PinHeader_2.54mm:PinHeader_1x02_P2.54mm_Vertical, F.Cu at (178.4, 113.7)
- added J25: R_Home_SW, Connector_PinHeader_2.54mm:PinHeader_1x02_P2.54mm_Vertical, F.Cu at (178.4, 136.5)
- added R2: 10k, Resistor_SMD:R_0805_2012Metric_Pad1.20x1.40mm_HandSolder, F.Cu at (185.4, 79.4)
- added R3: 10k, Resistor_SMD:R_0805_2012Metric_Pad1.20x1.40mm_HandSolder, F.Cu at (185.4, 125.1)
- added R4: 10k, Resistor_SMD:R_0805_2012Metric_Pad1.20x1.40mm_HandSolder, F.Cu at (185.4, 102.2)
- added R5: 10k, Resistor_SMD:R_0805_2012Metric_Pad1.20x1.40mm_HandSolder, F.Cu at (185.4, 90.8)
- added R6: 10k, Resistor_SMD:R_0805_2012Metric_Pad1.20x1.40mm_HandSolder, F.Cu at (185.4, 136.5)
- added R7: 10k, Resistor_SMD:R_0805_2012Metric_Pad1.20x1.40mm_HandSolder, F.Cu at (185.4, 113.7)
- added SW2: Y_Enable, Button_Switch_THT:SW_CuK_OS102011MA1QN1_SPDT_Angled, F.Cu at (191.0, 107.4)
- added SW3: A1_Enable, Button_Switch_THT:SW_CuK_OS102011MA1QN1_SPDT_Angled, F.Cu at (191.0, 96.0)
- added SW4: Z_Enable, Button_Switch_THT:SW_CuK_OS102011MA1QN1_SPDT_Angled, F.Cu at (191.0, 130.3)
- added SW5: A2_Enable, Button_Switch_THT:SW_CuK_OS102011MA1QN1_SPDT_Angled, F.Cu at (191.0, 118.8)
- added SW6: R_Enable, Button_Switch_THT:SW_CuK_OS102011MA1QN1_SPDT_Angled, F.Cu at (191.0, 141.7)
- R1: value 120 -> 290
- SW1: value SW_SPDT -> X_Enable
- moved SW1 96.2 mm to (191.0, 84.5), turned to 90 degrees
- moved U2 20.6 mm to (156.2, 170.8), turned to -90 degrees
- moved D1 20.1 mm to (158.0, 156.2)
- moved R1 20.1 mm to (164.7, 156.2)
- moved C1 18.1 mm to (153.7, 163.8), turned to 90 degrees
- moved J13 17.8 mm to (139.1, 161.7)
- moved U3 15.5 mm to (168.2, 170.6), turned to -90 degrees
- moved C2 11.5 mm to (158.8, 163.8), turned to -90 degrees
- moved J1 9.92 mm to (170.8, 80.6)
- moved J4 9.44 mm to (170.8, 92.1)
- moved C4 9.03 mm to (170.8, 163.8), turned to -90 degrees
- moved J2 8.98 mm to (170.8, 103.5)
- moved J5 8.53 mm to (170.8, 115.0)
- moved J3 8.13 mm to (170.8, 126.4)
- moved J6 7.75 mm to (170.8, 137.8)
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Connections:
- C2 pad 2: /24V_Toggle -> +24V
- C3 pad 2: Net-(U3-GND) -> GND
- C4 pad 1: Net-(U3-GND) -> GND
- C4 pad 2: /24V_Toggle -> +24V
- D1 pad 2: +3.3V -> +5V
- J1 pad 3: /X_Home -> Net-(J1-Pin_3)
- J10 pad 1: +5V -> /A1_B
- J10 pad 2: /A2_A -> +5V
- J10 pad 3: /A2_B -> /A1_A
- J11 pad 1: +5V -> /A2_B
- J11 pad 2: /A1_A -> +5V
- J11 pad 3: /A1_B -> /A2_A
- J12 pad 1: +5V -> /R_B
- J12 pad 2: /R_A -> +5V
- J12 pad 3: /R_B -> /R_A
- J14 pad 1: /24V_Toggle -> +24V
- J15 pad 1: /24V_Toggle -> +24V
- J16 pad 1: /24V_Toggle -> +24V
- J17 pad 1: /24V_Toggle -> +24V
- J18 pad 1: /24V_Toggle -> +24V
- J19 pad 1: /24V_Toggle -> +24V
- J2 pad 3: /Y_Home -> Net-(J2-Pin_3)
- J3 pad 3: /Z_Home -> Net-(J3-Pin_3)
- J4 pad 3: /A1_Home -> Net-(J4-Pin_3)
- J5 pad 3: /A2_Home -> Net-(J5-Pin_3)
- J6 pad 3: /R_Home -> Net-(J6-Pin_3)
- J7 pad 1: +5V -> /Y_B
- J7 pad 2: /Y_A -> +5V
- J7 pad 3: /Y_B -> /Y_A
- J8 pad 1: +5V -> /X_B
- J8 pad 2: /X_A -> +5V
- J8 pad 3: /X_B -> /X_A
- J9 pad 1: +5V -> /Z_B
- J9 pad 2: /Z_A -> +5V
- J9 pad 3: /Z_B -> /Z_A
- SW1 pad 1: /24V_Toggle -> +5V
- SW1 pad 2: +24V -> Net-(J1-Pin_3)
- SW1 pad 3: unconnected-(SW1-C-Pad3) -> GND
- U1 pad CN6_4: unconnected-(U1C-CN6_+3V3-PadCN6_4) -> +3.3V
- U1 pad CN6_8: +3.3V -> unconnected-(U1C-CN6_VIN-PadCN6_8)
- U2 pad 1: /24V_Toggle -> +24V
- U3 pad 1: /24V_Toggle -> +24V
- U3 pad 2: Net-(U3-GND) -> GND
Routing:
- net /24V_Toggle: track 130.4 -> 0.00 mm
- net +24V: track 18.0 -> 102.4 mm, vias 0 -> 2
- net +3.3V: track 101.6 -> 183.7 mm, vias 2 -> 1
- net /X_Home: track 24.4 -> 55.8 mm, vias 1 -> 0
- net /A2_B: track 65.9 -> 38.1 mm
- net Net-(J5-Pin_3): track 0.00 -> 21.5 mm
- net Net-(J6-Pin_3): track 0.00 -> 21.5 mm
- net Net-(J4-Pin_3): track 0.00 -> 21.5 mm
- net Net-(J2-Pin_3): track 0.00 -> 21.5 mm
- net Net-(J1-Pin_3): track 0.00 -> 21.5 mm
- net Net-(J3-Pin_3): track 0.00 -> 21.5 mm
- net Net-(U3-GND): track 16.3 -> 0.00 mm
- net /A1_A: track 51.7 -> 65.7 mm
- net /Y_Home: track 20.0 -> 33.2 mm, vias 0 -> 1
- net +5V: track 6.17 -> 19.4 mm
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