Commit message: current test for basic server for interface with moveit

File: ros_workspaces/src/gantry_controller/config/gazebo_gantry.urdf (robot description, URDF)
Before this commit: robot gantry, 8 links, 7 joints
Joints:
- joint TMS_1: origin xyz=0.00034733 -0.00025 -0.34785 rpy=2.266 -0.99955 0.78967 -> xyz=0.00034733 -0.00025 -0.34785 rpy=0 0 0
- joint TMS_HEAD: origin xyz=0 0 0 rpy=1.3245 0.71549 -0.069725 -> xyz=0 0 0 rpy=0 0 0
