Commit message: put urdf into ros project

File: ros_workspaces/src/gantry/urdf/gantry.urdf (robot description, URDF)
Before this commit: robot gantry, 7 links, 6 joints
Links:
- removed link R_arm
- removed link TMS_1
- removed link TMS_HEAD
- removed link X_gantry
- removed link Y_gantry
- removed link Z_gantry
- added link R_arm_link, mass 0.408324104757072; collision mesh filename=package://gantry/meshes/R_arm.STL; visual mesh filename=package://gantry/meshes/R_arm.STL
- added link TMS_1_link, mass 0.0116350451938087; collision mesh filename=package://gantry/meshes/TMS_1.STL; visual mesh filename=package://gantry/meshes/TMS_1.STL
- added link TMS_HEAD_link, mass 0.0428411645602252; collision mesh filename=package://gantry/meshes/TMS_HEAD.STL; visual mesh filename=package://gantry/meshes/TMS_HEAD.STL
- added link X_gantry_link, mass 2.7184408688585; collision mesh filename=package://gantry/meshes/X_gantry.STL; visual mesh filename=package://gantry/meshes/X_gantry.STL
- added link Y_gantry_link, mass 1.32530018007877; collision mesh filename=package://gantry/meshes/Y_gantry.STL; visual mesh filename=package://gantry/meshes/Y_gantry.STL
- added link Z_gantry_link, mass 0.403068685283753; collision mesh filename=package://gantry/meshes/Z_gantry.STL; visual mesh filename=package://gantry/meshes/Z_gantry.STL
Joints:
- joint R_arm: child R_arm -> R_arm_link; parent Z_gantry -> Z_gantry_link
- joint TMS_1: child TMS_1 -> TMS_1_link; parent R_arm -> R_arm_link
- joint TMS_HEAD: child TMS_HEAD -> TMS_HEAD_link; parent TMS_1 -> TMS_1_link
- joint X_gantry: child X_gantry -> X_gantry_link
- joint Y_gantry: child Y_gantry -> Y_gantry_link; parent X_gantry -> X_gantry_link
- joint Z_gantry: child Z_gantry -> Z_gantry_link; parent Y_gantry -> Y_gantry_link

Commit message: Robot is now in MoveIt

File: ros_workspaces/src/gantry/urdf/gantry.urdf (robot description, URDF)
Before this commit: robot gantry, 7 links, 6 joints
Links:
- added link world
Joints:
- added joint base_joint: type fixed, parent world, child base_link, origin xyz=0.0 0.0 0.17 rpy=0 0 0
- joint X_gantry: limit lower=0 upper=0 effort=0 velocity=0 -> lower=-0.28 upper=0 effort=0 velocity=0
- joint Y_gantry: limit lower=0 upper=0 effort=0 velocity=0 -> lower=0 upper=0.16 effort=0 velocity=0
- joint Z_gantry: limit lower=0 upper=0 effort=0 velocity=0 -> lower=-0.03 upper=0.1 effort=0 velocity=0

Commit message: new URDF

File: ros_workspaces/src/gantry/urdf/gantry.urdf (robot description, URDF)
Before this commit: robot gantry, 8 links, 7 joints
Links:
- removed link R_arm_link
- removed link TMS_1_link
- removed link TMS_HEAD_link
- removed link X_gantry_link
- removed link Y_gantry_link
- removed link Z_gantry_link
- removed link world
- added link R_Arm_Link, mass 0.645326600445391; collision mesh filename=package://gantry/meshes/R_Arm_Link.STL; visual mesh filename=package://gantry/meshes/R_Arm_Link.STL
- added link TMS_1_Link, mass 0.0116350451938088; collision mesh filename=package://gantry/meshes/TMS_1_Link.STL; visual mesh filename=package://gantry/meshes/TMS_1_Link.STL
- added link TMS_HEAD_Link, mass 0.0428412061325881; collision mesh filename=package://gantry/meshes/TMS_HEAD_Link.STL; visual mesh filename=package://gantry/meshes/TMS_HEAD_Link.STL
- added link X_Gantry_Link, mass 2.7184408688585; collision mesh filename=package://gantry/meshes/X_Gantry_Link.STL; visual mesh filename=package://gantry/meshes/X_Gantry_Link.STL
- added link Y_Gantry_Link, mass 1.32530018007878; collision mesh filename=package://gantry/meshes/Y_Gantry_Link.STL; visual mesh filename=package://gantry/meshes/Y_Gantry_Link.STL
- added link Z_Gantry_Link, mass 0.403068685283753; collision mesh filename=package://gantry/meshes/Z_Gantry_Link.STL; visual mesh filename=package://gantry/meshes/Z_Gantry_Link.STL
- link base_link: mass 0.999102566758599 -> 0.999102566760147
Joints:
- removed joint R_arm
- removed joint X_gantry
- removed joint Y_gantry
- removed joint Z_gantry
- removed joint base_joint
- added joint R_Arm: type continuous, parent Z_Gantry_Link, child R_Arm_Link, origin xyz=-0.0535 -0.10003 -0.0569 rpy=3.1416 0 3.1416, axis 1 0 0
- added joint Y_Gantry: type prismatic, parent X_Gantry_Link, child Y_Gantry_Link, origin xyz=-0.242 0.462 -0.1655 rpy=0 0 0, axis 0 -1 0, limit lower=-0.16 upper=0 effort=0 velocity=0
- added joint Z_Gantry: type prismatic, parent Y_Gantry_Link, child Z_Gantry_Link, origin xyz=-0.046503 -0.079468 -0.059 rpy=0 0 0, axis 0 0 1, limit lower=0 upper=0.13 effort=0 velocity=0
- added joint x_Gantry: type prismatic, parent base_link, child X_Gantry_Link, origin xyz=0.067498 0.0425 0.0225 rpy=1.5708 0 -1.5708, axis -1 0 0, limit lower=0 upper=0.3 effort=0 velocity=0
- joint TMS_1: axis 0.38068 0 0.92471 -> 0 1 0; child TMS_1_link -> TMS_1_Link; origin xyz=0.00034733 -0.00025 -0.34785 rpy=2.266 -0.99955 0.78967 -> xyz=0.000347 0.07525 0.3706 rpy=1.5708 0 0; parent R_arm_link -> R_Arm_Link
- joint TMS_HEAD: axis 0.85728 0.37485 -0.35292 -> 1 0 0; child TMS_HEAD_link -> TMS_HEAD_Link; origin xyz=0 0 0 rpy=1.3245 0.71549 -0.069725 -> xyz=0 0 0 rpy=0 0 3.1416; parent TMS_1_link -> TMS_1_Link

Commit message: stuff

File: ros_workspaces/src/gantry/urdf/gantry.urdf (robot description, URDF)
Before this commit: robot gantry, 7 links, 6 joints
Links:
- link R_Arm_Link: mass 0.645326600445391 -> 0.64532660044539
- link TMS_HEAD_Link: mass 0.0428412061325881 -> 0.0428412061326084
- link Z_Gantry_Link: mass 0.403068685283753 -> 0.403068685283752
Joints:
- joint R_Arm: axis 1 0 0 -> 0 0 1; origin xyz=-0.0535 -0.10003 -0.0569 rpy=3.1416 0 3.1416 -> xyz=-0.0534999999999979 -0.100032269904372 -0.0569000000000014 rpy=3.14159265358979 0 3.14159265358979
- joint TMS_1: axis 0 1 0 -> 1 0 0; origin xyz=0.000347 0.07525 0.3706 rpy=1.5708 0 0 -> xyz=0.000346999570831286 0.0752500000000218 0.370600000000016 rpy=1.57079632679489 0 0
- joint TMS_HEAD: axis 1 0 0 -> 0 0 1; origin xyz=0 0 0 rpy=0 0 3.1416 -> xyz=0 0 0 rpy=0 0 3.14159265358979
- joint Y_Gantry: axis 0 -1 0 -> 1 0 0; origin xyz=-0.242 0.462 -0.1655 rpy=0 0 0 -> xyz=-0.241997500000031 0.461999999999982 -0.165502499998546 rpy=0 0 0
- joint Z_Gantry: axis 0 0 1 -> 0 1 0; origin xyz=-0.046503 -0.079468 -0.059 rpy=0 0 0 -> xyz=-0.0465025000000195 -0.0794677300954897 -0.0589999999999941 rpy=0 0 0
- joint x_Gantry: axis -1 0 0 -> 0 0 1; origin xyz=0.067498 0.0425 0.0225 rpy=1.5708 0 -1.5708 -> xyz=0.0674975000000973 0.0424999999999915 0.0224999999999924 rpy=1.5707963267949 0 -1.5707963267949

Commit message: updated URDF file

File: ros_workspaces/src/gantry/urdf/gantry.urdf (robot description, URDF)
Before this commit: robot gantry, 7 links, 6 joints
Joints:
- joint Y_Gantry: limit lower=-0.16 upper=0 effort=0 velocity=0 -> lower=0 upper=0.169 effort=0 velocity=0
- joint Z_Gantry: limit lower=0 upper=0.13 effort=0 velocity=0 -> lower=-0.137 upper=0 effort=0 velocity=0
- joint x_Gantry: limit lower=0 upper=0.3 effort=0 velocity=0 -> lower=-0.3 upper=0 effort=0 velocity=0
